Commit message: Rotation of 180 deg on x axis for front_laser frame

File: my_rb1_description/urdf/my_rb1_robot.urdf (robot description, URDF)
Before this commit: robot rb1_robot, 7 links, 6 joints
Joints:
- joint base_link_front_laser_joint: origin xyz=0.25 0 0.075 rpy=0 0 0 -> xyz=0.25 0 0.075 rpy=3.1414 0 0

Commit message: Migrating materials, wheel friction and ROS Plugins

File: my_rb1_description/urdf/my_rb1_robot.urdf (robot description, URDF)
Before this commit: robot rb1_robot, 7 links, 6 joints
Links:
- link front_laser: geometry 
